Commit message: S

File: azrael_description/urdf/system.urdf.xacro (robot description, xacro)
@@ -76,3 +76,10 @@
     <axis xyz="0 0 1"/>
   </joint>
+  <link name="tcp" />
+  <joint name="$(arg prefix)tcpjoint" type="fixed">
+    <parent link="$(arg prefix)tool0"/>
+    <child link="tcp"/>
+    <origin xyz="-0.195 0 -0.3" rpy=" 0 0 0"/>
+    <axis xyz="0 0 1"/>
+  </joint>
 </robot>

Commit message: S

File: azrael_description/urdf/system.urdf.xacro (robot description, xacro)
@@ -80,5 +80,5 @@
     <parent link="$(arg prefix)tool0"/>
     <child link="tcp"/>
-    <origin xyz="-0.195 0 -0.3" rpy=" 0 0 0"/>
+    <origin xyz="-0.195 0 0.3" rpy=" 0 0 ${M_PI/2}"/>
     <axis xyz="0 0 1"/>
   </joint>

Commit message: tcp_fix

File: azrael_description/urdf/system.urdf.xacro (robot description, xacro)
@@ -80,5 +80,5 @@
     <parent link="$(arg prefix)tool0"/>
     <child link="tcp"/>
-    <origin xyz="-0.195 0 0.3" rpy=" 0 0 ${M_PI/2}"/>
+    <origin xyz="0.195 0 0.3" rpy=" 0 0 -${M_PI/2}"/>
     <axis xyz="0 0 1"/>
   </joint>

Commit message: tcp urdf

File: azrael_description/urdf/system.urdf.xacro (robot description, xacro)
@@ -80,5 +80,5 @@
     <parent link="$(arg prefix)tool0"/>
     <child link="tcp"/>
-    <origin xyz="0.195 0 0.3" rpy=" 0 0 -${M_PI/2}"/>
+    <origin xyz="0.08 0 0.33" rpy=" 0 0 -${M_PI/2}"/>
     <axis xyz="0 0 1"/>
   </joint>

Commit message: S

File: azrael_description/urdf/system.urdf.xacro (robot description, xacro)
@@ -1,4 +1,16 @@
 <?xml version="1.0"?>
 <robot name="tm12" xmlns:xacro="http://ros.org/wiki/xacro">
+  <material name="black">
+    <color rgba="0. 0. 0. 1" />
+  </material>
+  <material name="dark_grey">
+    <color rgba="0.1 0.1 0.1 1" />
+  </material>
+  <material name="grey">
+    <color rgba="0.6 0.6 0.6 1" />
+  </material>
+  <material name="white">
+    <color rgba="0.9 0.9 0.9 1" />
+  </material>
   <xacro:include filename="$(find azrael_description)/urdf/azrael/azrael.xacro" />
   <xacro:arg name="name" default="ur"/>
@@ -80,6 +92,50 @@
     <parent link="$(arg prefix)tool0"/>
     <child link="tcp"/>
-    <origin xyz="0.08 0 0.33" rpy=" 0 0 -${M_PI/2}"/>
+    <origin xyz="0.02 0.00 0.34" rpy=" 0 0 -${M_PI/2}"/>
     <axis xyz="0 0 1"/>
   </joint>
+  <!-- <link name="camera_base" /> -->
+  <joint name="$(arg prefix)tcpcamera" type="fixed">
+    <parent link="tcp"/>
+    <child link="camera_base"/>
+    <origin xyz="0 0.31 -0.707" rpy=" 3.14 -0.785 1.571"/>
+    <axis xyz="0 0 1"/>
+  </joint>
+  <link name="camera_body">
+    <visual>
+      <origin xyz="0. 0. 0." />
+      <geometry>
+        <box size="0.0994 0.0996 0.023" />
+      </geometry>
+      <material name="white" />
+    </visual>
+  </link>
+  <link name="camera_base">
+    <visual>
+      <origin xyz="-0.013 0. 0." />
+      <geometry>
+        <box size="0.026 0.103 0.039" />
+      </geometry>
+      <material name="grey" />
+    </visual>
+  </link>
+  <link name="camera_visor">
+    <visual>
+      <origin xyz="-0.0128 0. 0." />
+      <geometry>
+        <box size="0.026 0.101 0.037" />
+      </geometry>
+      <material name="black" />
+    </visual>
+  </link>
+  <joint name="camera_base_to_body" type="fixed">
+    <parent link="camera_base" />
+    <child link="camera_body" />
+    <origin xyz="-0.0757 0. 0.008" rpy="0. 0. 0." />
+  </joint>
+  <joint name="camera_base_to_visor" type="fixed">
+    <parent link="camera_base" />
+    <child link="camera_visor" />
+    <origin xyz="0. 0. 0." rpy="0. 0. 0." />
+  </joint>
 </robot>

Commit message: update xacro

File: azrael_description/urdf/system.urdf.xacro (robot description, xacro)
@@ -1,4 +1,4 @@
 <?xml version="1.0"?>
-<robot name="tm12" xmlns:xacro="http://ros.org/wiki/xacro">
+<robot name="azrael" xmlns:xacro="http://ros.org/wiki/xacro">
   <material name="black">
     <color rgba="0. 0. 0. 1" />
@@ -17,4 +17,6 @@
   <xacro:include filename="$(find azrael_description)/urdf/ur_macro.xacro"/>
   <xacro:arg name="ur_type" default="ur10"/>
+  <xacro:arg name="ft_sensor_ros2_control" default="false"/>
+  <xacro:arg name="gripper_ros2_control" default="false"/>
   <!-- parameters -->
   <xacro:arg name="prefix" default="" />
@@ -139,3 +141,13 @@
     <origin xyz="0. 0. 0." rpy="0. 0. 0." />
   </joint>
+  <xacro:include filename="$(find robotiq_ft_sensor_description)/urdf/robotiq_ft300s.urdf.xacro"/>
+  <xacro:include filename="$(find robotiq_description)/urdf/robotiq_2f_140_macro.urdf.xacro"/>
+  <xacro:robotiq_ft300s parent="tool0" tf_prefix="$(arg prefix)">
+    <origin xyz="0 0 -0.04875" rpy="0 0 0"/>
+  </xacro:robotiq_ft300s>
+  <xacro:robotiq_gripper name="azrael_gripper" prefix="$(arg prefix)" parent="$(arg prefix)robotiq_ft_frame_id" include_ros2_control="false">
+    <origin xyz="0 0 -0.00695" rpy="0 0 ${pi/2}"/>
+  </xacro:robotiq_gripper>
+  <xacro:include filename="tools.ros2_control.xacro"/>
+  <xacro:tools_ros2_control prefix="$(arg prefix)" ft_sensor="$(arg ft_sensor_ros2_control)" gripper="$(arg gripper_ros2_control)"/>
 </robot>

Commit message: misc

File: azrael_description/urdf/system.urdf.xacro (robot description, xacro)
@@ -20,6 +20,5 @@
   <xacro:arg name="gripper_ros2_control" default="false"/>
   <!-- parameters -->
-  <xacro:arg name="prefix" default="" />
-  <xacro:arg name="prefix_rc" default="" />
+  <xacro:arg name="prefix" default="az_" />
   <xacro:arg name="joint_limit_params" default="$(find azrael_description)/config/$(arg ur_type)/joint_limits.yaml"/>
   <xacro:arg name="kinematics_params" default="$(find azrael_description)/config/$(arg ur_type)/default_kinematics.yaml"/>
@@ -53,4 +52,5 @@
     <origin xyz="0 0 0" rpy="0 0 0" />
   </xacro:azrael>
+  <!-- <link name="$(arg prefix)base_footprint"/> -->
    <!-- arm -->
   <xacro:ur_robot
@@ -82,21 +82,15 @@
     robot_ip="$(arg robot_ip)"
     >
-    <origin xyz="0 0 0" rpy="0 0 0" />
+    <origin xyz="0.0 0.1 0.28" rpy="0 0 0"/>
   </xacro:ur_robot>
-  <joint name="$(arg prefix)lifter" type="fixed">
-    <parent link="$(arg prefix)base_footprint"/>
-    <child link="$(arg prefix)base_link"/>
-    <origin xyz="0.0 0.1 0.28" rpy=" 0 0 0"/>
-    <axis xyz="0 0 1"/>
-  </joint>
-  <link name="tcp" />
+  <link name="$(arg prefix)tcp" />
   <joint name="$(arg prefix)tcpjoint" type="fixed">
     <parent link="$(arg prefix)tool0"/>
-    <child link="tcp"/>
+    <child link="$(arg prefix)tcp"/>
     <origin xyz="0.02 0.00 0.34" rpy=" 0 0 -${M_PI/2}"/>
     <axis xyz="0 0 1"/>
   </joint>
   <!-- <link name="camera_base" /> -->
-  <joint name="$(arg prefix)tcpcamera" type="fixed">
+  <!-- <joint name="$(arg prefix)tcpcamera" type="fixed">
     <parent link="tcp"/>
     <child link="camera_base"/>
@@ -140,13 +134,13 @@
     <child link="camera_visor" />
     <origin xyz="0. 0. 0." rpy="0. 0. 0." />
-  </joint>
+  </joint> -->
   <xacro:include filename="$(find robotiq_ft_sensor_description)/urdf/robotiq_ft300s.urdf.xacro"/>
-  <xacro:include filename="$(find robotiq_description)/urdf/robotiq_2f_140_macro.urdf.xacro"/>
+  <!-- <xacro:include filename="$(find robotiq_description)/urdf/robotiq_2f_140_macro.urdf.xacro"/> -->
   <xacro:robotiq_ft300s parent="tool0" tf_prefix="$(arg prefix)">
-    <origin xyz="0 0 -0.04875" rpy="0 0 0"/>
+    <origin xyz="0 0 ${-6.5/1000}" rpy="0 0 0"/>
   </xacro:robotiq_ft300s>
-  <xacro:robotiq_gripper name="azrael_gripper" prefix="$(arg prefix)" parent="$(arg prefix)robotiq_ft_frame_id" include_ros2_control="false">
+  <!-- <xacro:robotiq_gripper name="azrael_gripper" prefix="$(arg prefix)" parent="$(arg prefix)robotiq_ft_frame_id" include_ros2_control="false">
     <origin xyz="0 0 -0.00695" rpy="0 0 ${pi/2}"/>
-  </xacro:robotiq_gripper>
+  </xacro:robotiq_gripper> -->
   <xacro:include filename="tools.ros2_control.xacro"/>
   <xacro:tools_ros2_control prefix="$(arg prefix)" ft_sensor="$(arg ft_sensor_ros2_control)" gripper="$(arg gripper_ros2_control)"/>

File: azrael_description/urdf/tools.ros2_control.xacro (robot description, xacro)
@@ -4,9 +4,9 @@
     <xacro:if value="${ft_sensor}">
       <xacro:include filename="$(find robotiq_ft_sensor_description)/urdf/robotiq_fts.ros2_control.xacro"/>
-      <xacro:robotiq_fts_ros2_control name="${prefix}omron_imm/" tf_prefix="${prefix}"/>
+      <xacro:robotiq_fts_ros2_control name="${prefix}" tf_prefix="${prefix}"/>
     </xacro:if>
     <xacro:if value="${gripper}">
       <xacro:include filename="$(find robotiq_description)/urdf/2f_140.ros2_control.xacro"/>
-      <xacro:robotiq_gripper_ros2_control name="${prefix}omron_imm/robotiq_2f_140" prefix="${prefix}"/>
+      <xacro:robotiq_gripper_ros2_control name="${prefix}robotiq_2f_140" prefix="${prefix}"/>
     </xacro:if>
   </xacro:macro>

File: azrael_description/urdf/ur.ros2_control.xacro (robot description, xacro)
@@ -24,5 +24,5 @@
           <param name="reverse_port">${reverse_port}</param>
           <param name="script_sender_port">${script_sender_port}</param>
-          <param name="tf_prefix">"${tf_prefix}"</param>
+          <param name="tf_prefix">${tf_prefix}</param>
           <param name="non_blocking_read">0</param>
           <param name="servoj_gain">2000</param>
@@ -39,4 +39,7 @@
           <param name="tool_tcp_port">${tool_tcp_port}</param>
         </xacro:unless>
+        <xacro:if value="${use_fake_hardware}">
+          <plugin>mock_components/GenericSystem</plugin>
+        </xacro:if>
       </hardware>
       <joint name="${prefix}shoulder_pan_joint">
@@ -146,5 +149,5 @@
         </sensor>
         <!-- NOTE The following are joints used only for testing with fake hardware and will change in the future -->
-        <gpio name="speed_scaling">
+        <!-- <gpio name="speed_scaling">
           <state_interface name="speed_scaling_factor"/>
           <param name="initial_speed_scaling_factor">1</param>
@@ -258,5 +261,5 @@
         <gpio name="system_interface">
           <state_interface name="initialized"/>
-        </gpio>
+        </gpio> -->
       </xacro:unless>
     </ros2_control>

File: azrael_description/urdf/ur_macro.xacro (robot description, xacro)
@@ -52,5 +52,5 @@
       sim_gazebo="${sim_gazebo}"
       sim_ignition="${sim_ignition}"
-      tf_prefix=""
+      tf_prefix="${prefix}"
       hash_kinematics="${kinematics_hash}"
       robot_ip="${robot_ip}"

Commit message: add fake ft sensor

File: azrael_description/urdf/system.urdf.xacro (robot description, xacro)
@@ -144,4 +144,4 @@
   </xacro:robotiq_gripper> -->
   <xacro:include filename="tools.ros2_control.xacro"/>
-  <xacro:tools_ros2_control prefix="$(arg prefix)" ft_sensor="$(arg ft_sensor_ros2_control)" gripper="$(arg gripper_ros2_control)"/>
+  <xacro:tools_ros2_control prefix="$(arg prefix)" ft_sensor="$(arg ft_sensor_ros2_control)" gripper="$(arg gripper_ros2_control)" ft_sensor_fake="$(arg use_fake_hardware)"/>
 </robot>

File: azrael_description/urdf/tools.ros2_control.xacro (robot description, xacro)
@@ -1,8 +1,11 @@
 <?xml version="1.0"?>
 <robot xmlns:xacro="http://www.ros.org/wiki/xacro">
-  <xacro:macro name="tools_ros2_control" params="prefix ft_sensor gripper">
+  <xacro:macro name="tools_ros2_control" params="prefix
+                                                 ft_sensor
+                                                 gripper
+                                                 ft_sensor_fake:=false">
     <xacro:if value="${ft_sensor}">
       <xacro:include filename="$(find robotiq_ft_sensor_description)/urdf/robotiq_fts.ros2_control.xacro"/>
-      <xacro:robotiq_fts_ros2_control name="${prefix}" tf_prefix="${prefix}"/>
+      <xacro:robotiq_fts_ros2_control name="${prefix}" tf_prefix="${prefix}" use_fake_mode="${ft_sensor_fake}"/>
     </xacro:if>
     <xacro:if value="${gripper}">

Commit message: clean urdf

File: azrael_description/urdf/system.urdf.xacro (robot description, xacro)
@@ -17,6 +17,4 @@
   <xacro:include filename="$(find azrael_description)/urdf/ur_macro.xacro"/>
   <xacro:arg name="ur_type" default="ur10"/>
-  <xacro:arg name="ft_sensor_ros2_control" default="false"/>
-  <xacro:arg name="gripper_ros2_control" default="false"/>
   <!-- parameters -->
   <xacro:arg name="prefix" default="az_" />
@@ -62,5 +60,5 @@
     physical_parameters_file="$(arg physical_params)"
     visual_parameters_file="$(arg visual_params)"
-    initial_positions="${dict(shoulder_pan_joint=0.0,shoulder_lift_joint=-2.3,elbow_joint=1.7,wrist_1_joint=-2.57,wrist_2_joint=0.5,wrist_3_joint=0.0)}"
+    initial_positions="${dict(shoulder_pan_joint=0.0,shoulder_lift_joint=-2.70,elbow_joint=2.26,wrist_1_joint=-0.43,wrist_2_joint=0.5,wrist_3_joint=0.0)}"
     transmission_hw_interface="$(arg transmission_hw_interface)"
     safety_limits="$(arg safety_limits)"
@@ -85,64 +83,10 @@
     <origin xyz="0.0 0.1 0.28" rpy="0 0 0"/>
   </xacro:ur_robot>
-  <link name="$(arg prefix)tcp" />
+<!--  <link name="$(arg prefix)tcp" />
   <joint name="$(arg prefix)tcpjoint" type="fixed">
     <parent link="$(arg prefix)tool0"/>
     <child link="$(arg prefix)tcp"/>
-    <origin xyz="0.02 0.00 0.34" rpy=" 0 0 -${M_PI/2}"/>
+    <origin xyz="0.0 0.00 0.34" rpy=" 0 0 -${M_PI/2}"/>
     <axis xyz="0 0 1"/>
-  </joint>
-  <!-- <link name="camera_base" /> -->
-  <!-- <joint name="$(arg prefix)tcpcamera" type="fixed">
-    <parent link="tcp"/>
-    <child link="camera_base"/>
-    <origin xyz="0 0.31 -0.707" rpy=" 3.14 -0.785 1.571"/>
-    <axis xyz="0 0 1"/>
-  </joint>
-  <link name="camera_body">
-    <visual>
-      <origin xyz="0. 0. 0." />
-      <geometry>
-        <box size="0.0994 0.0996 0.023" />
-      </geometry>
-      <material name="white" />
-    </visual>
-  </link>
-  <link name="camera_base">
-    <visual>
-      <origin xyz="-0.013 0. 0." />
-      <geometry>
-        <box size="0.026 0.103 0.039" />
-      </geometry>
-      <material name="grey" />
-    </visual>
-  </link>
-  <link name="camera_visor">
-    <visual>
-      <origin xyz="-0.0128 0. 0." />
-      <geometry>
-        <box size="0.026 0.101 0.037" />
-      </geometry>
-      <material name="black" />
-    </visual>
-  </link>
-  <joint name="camera_base_to_body" type="fixed">
-    <parent link="camera_base" />
-    <child link="camera_body" />
-    <origin xyz="-0.0757 0. 0.008" rpy="0. 0. 0." />
-  </joint>
-  <joint name="camera_base_to_visor" type="fixed">
-    <parent link="camera_base" />
-    <child link="camera_visor" />
-    <origin xyz="0. 0. 0." rpy="0. 0. 0." />
-  </joint> -->
-  <xacro:include filename="$(find robotiq_ft_sensor_description)/urdf/robotiq_ft300s.urdf.xacro"/>
-  <!-- <xacro:include filename="$(find robotiq_description)/urdf/robotiq_2f_140_macro.urdf.xacro"/> -->
-  <xacro:robotiq_ft300s parent="tool0" tf_prefix="$(arg prefix)">
-    <origin xyz="0 0 ${-6.5/1000}" rpy="0 0 0"/>
-  </xacro:robotiq_ft300s>
-  <!-- <xacro:robotiq_gripper name="azrael_gripper" prefix="$(arg prefix)" parent="$(arg prefix)robotiq_ft_frame_id" include_ros2_control="false">
-    <origin xyz="0 0 -0.00695" rpy="0 0 ${pi/2}"/>
-  </xacro:robotiq_gripper> -->
-  <xacro:include filename="tools.ros2_control.xacro"/>
-  <xacro:tools_ros2_control prefix="$(arg prefix)" ft_sensor="$(arg ft_sensor_ros2_control)" gripper="$(arg gripper_ros2_control)" ft_sensor_fake="$(arg use_fake_hardware)"/>
+  </joint>-->
 </robot>

Commit message: wip

File: azrael_description/urdf/system.urdf.xacro (robot description, xacro)
@@ -18,5 +18,5 @@
   <xacro:arg name="ur_type" default="ur10"/>
   <!-- parameters -->
-  <xacro:arg name="prefix" default="az_" />
+  <xacro:arg name="prefix" default="azrael/" />
   <xacro:arg name="joint_limit_params" default="$(find azrael_description)/config/$(arg ur_type)/joint_limits.yaml"/>
   <xacro:arg name="kinematics_params" default="$(find azrael_description)/config/$(arg ur_type)/default_kinematics.yaml"/>
@@ -60,5 +60,5 @@
     physical_parameters_file="$(arg physical_params)"
     visual_parameters_file="$(arg visual_params)"
-    initial_positions="${dict(shoulder_pan_joint=0.0,shoulder_lift_joint=-2.70,elbow_joint=2.26,wrist_1_joint=-0.43,wrist_2_joint=0.5,wrist_3_joint=0.0)}"
+    initial_positions="${dict(shoulder_pan_joint=1.0,shoulder_lift_joint=-2.30,elbow_joint=2.26,wrist_1_joint=-0.43,wrist_2_joint=0.75,wrist_3_joint=0.0)}"
     transmission_hw_interface="$(arg transmission_hw_interface)"
     safety_limits="$(arg safety_limits)"
@@ -82,4 +82,5 @@
     >
     <origin xyz="0.0 0.1 0.28" rpy="0 0 0"/>
+<!--    <origin xyz="0.0 0.0 0.28" rpy="0 0 0"/>-->
   </xacro:ur_robot>
 <!--  <link name="$(arg prefix)tcp" />

File: azrael_description/urdf/ur_macro.xacro (robot description, xacro)
@@ -2,5 +2,5 @@
 <robot xmlns:xacro="http://wiki.ros.org/xacro">
   <xacro:include filename="$(find ur_description)/urdf/inc/ur_transmissions.xacro" />
-  <xacro:include filename="$(find ur_description)/urdf/inc/ur_common.xacro" />
+  <xacro:include filename="$(find azrael_description)/urdf/ur_common.xacro" />
   <xacro:macro name="ur_robot" params="
     name

Commit message: rotate base_footprint

File: azrael_description/urdf/system.urdf.xacro (robot description, xacro)
@@ -64,5 +64,5 @@
   <xacro:property name="M_PI" value="3.14159"/>
   <xacro:azrael  prefix="$(arg prefix)">
-    <origin xyz="0 0 0" rpy="0 0 0" />
+    <origin xyz="0 0 0" rpy="0 0 -${M_PI/2}" />
   </xacro:azrael>
   <!-- <link name="$(arg prefix)base_footprint"/> -->

Commit message: rotate ur

File: azrael_description/urdf/system.urdf.xacro (robot description, xacro)
@@ -107,5 +107,5 @@
     non_blocking_read="$(arg non_blocking_read)"
     keep_alive_count="$(arg keep_alive_count)">
-    <origin xyz="0.0 0.1 0.28" rpy="0 0 0" />          <!-- position robot in the world -->
+    <origin xyz="0.0 0.1 0.28" rpy="0 0 +${M_PI/2}" />          <!-- position robot in the world -->
    </xacro:ur_robot>
 <!--  <link name="$(arg prefix)tcp" />

Commit message: rotate ur

File: azrael_description/urdf/system.urdf.xacro (robot description, xacro)
@@ -107,5 +107,5 @@
     non_blocking_read="$(arg non_blocking_read)"
     keep_alive_count="$(arg keep_alive_count)">
-    <origin xyz="0.0 0.1 0.28" rpy="0 0 +${M_PI/2}" />          <!-- position robot in the world -->
+    <origin xyz="0.0 0.1 0.28" rpy="0 0 -${M_PI/2}" />          <!-- position robot in the world -->
    </xacro:ur_robot>
 <!--  <link name="$(arg prefix)tcp" />

Commit message: Readme and gripper

File: azrael_description/urdf/system.urdf.xacro (robot description, xacro)
@@ -109,4 +109,15 @@
     <origin xyz="0.0 0.1 0.28" rpy="0 0 0" />          <!-- position robot in the world -->
    </xacro:ur_robot>
+    <!-- Robotiq 2f-140 -->
+    <xacro:include filename="$(find robotiq_description)/urdf/robotiq_2f_140_macro.urdf.xacro" />
+    <xacro:robotiq_gripper name="RobotiqGripperHardwareInterface" prefix="" parent="$(arg prefix)tool0" use_fake_hardware="$(arg fake_ur)" com_port="/dev/ttyUSB0">
+        <origin xyz="0 0 0" rpy="0 0 0" />
+    </xacro:robotiq_gripper>
+    <link name="$(arg prefix)tcp" />
+    <joint name="$(arg prefix)tcpjoint" type="fixed">
+      <parent link="$(arg prefix)tool0"/>
+      <child link="$(arg prefix)tcp"/>
+        <origin xyz="0 0 0.15" rpy="0 0 0"/>
+    </joint>
 <!--  <link name="$(arg prefix)tcp" />
   <joint name="$(arg prefix)tcpjoint" type="fixed">

Commit message: Gripper and nav2 fixes

File: azrael_description/urdf/system.urdf.xacro (robot description, xacro)
@@ -109,4 +109,16 @@
     <origin xyz="0.0 0.1 0.28" rpy="0 0 -${M_PI/2}" />          <!-- position robot in the world -->
    </xacro:ur_robot>
+    <!-- Robotiq 2f-140 -->
+    <xacro:include filename="$(find robotiq_description)/urdf/robotiq_2f_140_macro.urdf.xacro" />
+    <xacro:robotiq_gripper name="RobotiqGripperHardwareInterface" prefix="" parent="$(arg prefix)tool0" use_fake_hardware="$(arg fake_ur)" com_port="/dev/ttyUSB1">
+        <origin xyz="0 0 0" rpy="0 0 0" />
+    </xacro:robotiq_gripper>
+    <link name="$(arg prefix)tcp" />
+    <joint name="$(arg prefix)tcpjoint" type="fixed">
+      <parent link="$(arg prefix)tool0"/>
+      <child link="$(arg prefix)tcp"/>
+        <origin xyz="0 0 0.15" rpy="0 0 0"/>
+    </joint>
+    <!-- Robotiq 2f-140 -->
 <!--  <link name="$(arg prefix)tcp" />
   <joint name="$(arg prefix)tcpjoint" type="fixed">

Commit message: Removed gripper

File: azrael_description/urdf/system.urdf.xacro (robot description, xacro)
@@ -110,5 +110,5 @@
    </xacro:ur_robot>
     <!-- Robotiq 2f-140 -->
-    <xacro:include filename="$(find robotiq_description)/urdf/robotiq_2f_140_macro.urdf.xacro" />
+    <!-- <xacro:include filename="$(find robotiq_description)/urdf/robotiq_2f_140_macro.urdf.xacro" />
     <xacro:robotiq_gripper name="RobotiqGripperHardwareInterface" prefix="" parent="$(arg prefix)tool0" use_fake_hardware="$(arg fake_ur)" com_port="/dev/ttyUSB1">
         <origin xyz="0 0 0" rpy="0 0 0" />
@@ -119,5 +119,5 @@
       <child link="$(arg prefix)tcp"/>
         <origin xyz="0 0 0.15" rpy="0 0 0"/>
-    </joint>
+    </joint> -->
 <!--  <link name="$(arg prefix)tcp" />
   <joint name="$(arg prefix)tcpjoint" type="fixed">

Commit message: add ur gpio controller + hack fix ur controller rate

File: azrael_description/urdf/system.urdf.xacro (robot description, xacro)
@@ -17,4 +17,5 @@
   <xacro:arg name="name" default="ur"/>
   <xacro:arg name="ur_type" default="ur10e"/>
+  <xacro:arg name="use_gripper" default="true"/>
   <!-- parameters -->
   <xacro:arg name="prefix" default="azrael/" />
@@ -107,17 +108,19 @@
     non_blocking_read="$(arg non_blocking_read)"
     keep_alive_count="$(arg keep_alive_count)">
-    <origin xyz="0.0 0.1 0.28" rpy="0 0 -${M_PI/2}" />          <!-- position robot in the world -->
+    <origin xyz="0.0 0.0 0.28" rpy="0 0 -${M_PI/2}" />          <!-- position robot in the world -->
    </xacro:ur_robot>
     <!-- Robotiq 2f-85 -->
-    <xacro:include filename="$(find robotiq_description)/urdf/robotiq_2f_85_macro.urdf.xacro" />
-    <xacro:robotiq_gripper name="RobotiqGripperHardwareInterface" prefix="" parent="$(arg prefix)tool0" use_fake_hardware="$(arg fake_ur)" com_port="/dev/ttyUSB1">
-        <origin xyz="0 0 0" rpy="0 0 0" />
-    </xacro:robotiq_gripper>
-    <link name="$(arg prefix)tcp" />
-    <joint name="$(arg prefix)tcpjoint" type="fixed">
-      <parent link="$(arg prefix)tool0"/>
-      <child link="$(arg prefix)tcp"/>
-        <origin xyz="0 0 0.15" rpy="0 0 0"/>
-    </joint>
+    <xacro:if value="$(arg use_gripper)">
+      <xacro:include filename="$(find robotiq_description)/urdf/robotiq_2f_85_macro.urdf.xacro" />
+      <xacro:robotiq_gripper name="RobotiqGripperHardwareInterface" prefix="" parent="$(arg prefix)tool0" use_fake_hardware="$(arg fake_ur)" com_port="/dev/ttyUSB1">
+          <origin xyz="0 0 0" rpy="0 0 0" />
+      </xacro:robotiq_gripper>
+      <link name="$(arg prefix)tcp" />
+      <joint name="$(arg prefix)tcpjoint" type="fixed">
+        <parent link="$(arg prefix)tool0"/>
+        <child link="$(arg prefix)tcp"/>
+          <origin xyz="0 0 0.15" rpy="0 0 0"/>
+      </joint>
+    </xacro:if>
     <!-- Robotiq 2f-85 -->
 <!--  <link name="$(arg prefix)tcp" />
