Commit message: add gripper to urdf

File: azrael_description/urdf/system.urdf.xacro (robot description, xacro)
@@ -17,5 +17,6 @@
   <xacro:arg name="name" default="ur"/>
   <xacro:arg name="ur_type" default="ur10e"/>
-  <xacro:arg name="use_gripper" default="true"/>
+  <xacro:arg name="gripper" default="None"/>
+  <xacro:property name="gripper" value="$(arg gripper)"/>
   <!-- parameters -->
   <xacro:arg name="prefix" default="azrael/" />
@@ -111,7 +112,9 @@
    </xacro:ur_robot>
     <!-- Robotiq 2f-85 -->
-    <xacro:if value="$(arg use_gripper)">
+    <xacro:if value="${gripper == 'robotiq-2f-85'}">
+      <xacro:include filename="$(find robotiq_description)/urdf/ur_to_robotiq_adapter.urdf.xacro"/>
       <xacro:include filename="$(find robotiq_description)/urdf/robotiq_2f_85_macro.urdf.xacro" />
-      <xacro:robotiq_gripper name="RobotiqGripperHardwareInterface" prefix="" parent="$(arg prefix)tool0" use_fake_hardware="$(arg fake_ur)" com_port="/dev/ttyUSB1">
+      <xacro:ur_to_robotiq prefix="$(arg prefix)" parent="$(arg prefix)tool0" child="$(arg prefix)mount_to_robotiq" rotation="${M_PI}"/>
+      <xacro:robotiq_gripper name="RobotiqGripperHardwareInterface" prefix="$(arg prefix)" parent="$(arg prefix)mount_to_robotiq" use_fake_hardware="$(arg fake_ur)" com_port="/dev/ttyUSB1">
           <origin xyz="0 0 0" rpy="0 0 0" />
       </xacro:robotiq_gripper>
@@ -120,14 +123,20 @@
         <parent link="$(arg prefix)tool0"/>
         <child link="$(arg prefix)tcp"/>
-          <origin xyz="0 0 0.15" rpy="0 0 0"/>
+          <origin xyz="0 0 0.171" rpy="0 0 0"/>
       </joint>
     </xacro:if>
-    <!-- Robotiq 2f-85 -->
-<!--  <link name="$(arg prefix)tcp" />
-  <joint name="$(arg prefix)tcpjoint" type="fixed">
-    <parent link="$(arg prefix)tool0"/>
-    <child link="$(arg prefix)tcp"/>
-    <origin xyz="0.0 0.00 0.34" rpy=" 0 0 -${M_PI/2}"/>
-    <axis xyz="0 0 1"/>
-  </joint>-->
+    <xacro:if value="${gripper == 'robotiq-2f-140'}">
+      <xacro:include filename="$(find robotiq_description)/urdf/ur_to_robotiq_adapter.urdf.xacro"/>
+      <xacro:include filename="$(find robotiq_description)/urdf/robotiq_2f_140_macro.urdf.xacro" />
+      <xacro:ur_to_robotiq prefix="$(arg prefix)" parent="$(arg prefix)tool0" child="$(arg prefix)mount_to_robotiq" rotation="${M_PI}"/>
+      <xacro:robotiq_gripper name="RobotiqGripperHardwareInterface" prefix="$(arg prefix)" parent="$(arg prefix)mount_to_robotiq" use_fake_hardware="$(arg fake_ur)" com_port="/dev/ttyUSB1">
+          <origin xyz="0 0 0" rpy="0 0 0" />
+      </xacro:robotiq_gripper>
+      <link name="$(arg prefix)tcp" />
+      <joint name="$(arg prefix)tcpjoint" type="fixed">
+        <parent link="$(arg prefix)tool0"/>
+        <child link="$(arg prefix)tcp"/>
+          <origin xyz="0 0 0.241" rpy="0 0 0"/>
+      </joint>
+    </xacro:if>
 </robot>
