Commit message: S

File: azrael_description/urdf/azrael/azrael.xacro (robot description, xacro)
@@ -53,5 +53,5 @@
     <link name="${prefix}laser" />
     <joint name="${prefix}laser_joint" type="fixed">
-      <origin xyz="0.0 0.56 0.3" rpy="0 0 -${M_PI/2}" />
+      <origin xyz="0.0 -0.65 0.3" rpy="0 0 -${M_PI/2}" />
       <parent link="${prefix}base_link_azrael" />
       <child link="${prefix}laser" />

Commit message: S

File: azrael_description/urdf/azrael/azrael.xacro (robot description, xacro)
@@ -53,5 +53,6 @@
     <link name="${prefix}laser" />
     <joint name="${prefix}laser_joint" type="fixed">
-      <origin xyz="0.0 -0.65 0.3" rpy="0 0 -${M_PI/2}" />
+      <!-- <origin xyz="0.0 -0.65 0.3" rpy="0 0 -${M_PI/2}" /> -->
+      <origin xyz="0.0 0.65 0.3" rpy="0 0 ${M_PI/2}" />
       <parent link="${prefix}base_link_azrael" />
       <child link="${prefix}laser" />

Commit message: S

File: azrael_description/urdf/azrael/azrael.xacro (robot description, xacro)
@@ -13,10 +13,4 @@
           <inertia ixx="0.001" ixy="0.01" ixz="0.01" iyy="0.001" iyz="0.01" izz="0.001" />
       </inertial>
-      <collision>
-        <origin xyz="0 0 0.005" rpy="0 0 0" />
-        <geometry>
-          <box size="${base_x_size} ${base_y_size} 0.01"/>
-        </geometry>
-      </collision>
     </link>
     <!-- Base link is the center of the robot's bottom plate -->
@@ -49,10 +43,9 @@
       <parent link="${prefix}base_footprint" />
       <child link="${prefix}base_link_azrael" />
-      <dynamics damping="0.7"/>
     </joint>
     <link name="${prefix}laser" />
     <joint name="${prefix}laser_joint" type="fixed">
       <!-- <origin xyz="0.0 -0.65 0.3" rpy="0 0 -${M_PI/2}" /> -->
-      <origin xyz="0.0 0.65 0.3" rpy="0 0 ${M_PI/2}" />
+      <origin xyz="0.65 0.0 0.3" rpy="0 0 0" />
       <parent link="${prefix}base_link_azrael" />
       <child link="${prefix}laser" />

File: azrael_description/urdf/system.urdf.xacro (robot description, xacro)
@@ -3,13 +3,13 @@
   <xacro:include filename="$(find azrael_description)/urdf/azrael/azrael.xacro" />
   <xacro:arg name="name" default="ur"/>
-  <xacro:include filename="$(find ur_description)/urdf/ur_macro.xacro"/>
+  <xacro:include filename="$(find azrael_description)/urdf/ur_macro.xacro"/>
   <xacro:arg name="ur_type" default="ur10"/>
   <!-- parameters -->
   <xacro:arg name="prefix" default="" />
   <xacro:arg name="prefix_rc" default="" />
-  <xacro:arg name="joint_limit_params" default="$(find ur_description)/config/$(arg ur_type)/joint_limits.yaml"/>
-  <xacro:arg name="kinematics_params" default="$(find ur_description)/config/$(arg ur_type)/default_kinematics.yaml"/>
-  <xacro:arg name="physical_params" default="$(find ur_description)/config/$(arg ur_type)/physical_parameters.yaml"/>
-  <xacro:arg name="visual_params" default="$(find ur_description)/config/$(arg ur_type)/visual_parameters.yaml"/>
+  <xacro:arg name="joint_limit_params" default="$(find azrael_description)/config/$(arg ur_type)/joint_limits.yaml"/>
+  <xacro:arg name="kinematics_params" default="$(find azrael_description)/config/$(arg ur_type)/default_kinematics.yaml"/>
+  <xacro:arg name="physical_params" default="$(find azrael_description)/config/$(arg ur_type)/physical_parameters.yaml"/>
+  <xacro:arg name="visual_params" default="$(find azrael_description)/config/$(arg ur_type)/visual_parameters.yaml"/>
   <xacro:arg name="transmission_hw_interface" default=""/>
   <xacro:arg name="safety_limits" default="false"/>
@@ -19,7 +19,4 @@
   <xacro:arg name="headless_mode" default="false" />
   <xacro:arg name="robot_ip" default="0.0.0.0" />
-  <xacro:arg name="script_filename" default=""/>
-  <xacro:arg name="output_recipe_filename" default=""/>
-  <xacro:arg name="input_recipe_filename" default=""/>
   <!--   tool communication related parameters-->
   <xacro:arg name="use_tool_communication" default="false" />
@@ -33,13 +30,9 @@
   <xacro:arg name="tool_tcp_port" default="54321" />
     <!-- Simulation parameters -->
-  <xacro:arg name="use_fake_hardware" default="true" />
+  <xacro:arg name="use_fake_hardware" default="false" />
   <xacro:arg name="fake_sensor_commands" default="false" />
   <xacro:arg name="sim_gazebo" default="false" />
   <xacro:arg name="sim_ignition" default="false" />
   <xacro:arg name="simulation_controllers" default="error_default" />
-  <!-- initial position for simulations (Fake Hardware, Gazebo, Ignition) -->
-  <xacro:arg name="initial_positions_file" default="$(find ur_description)/config/initial_positions.yaml"/>
-  <!-- convert to property to use substitution in function -->
-  <xacro:property name="initial_positions_file" default="$(arg initial_positions_file)"/>
   <xacro:property name="M_PI" value="3.14159"/>
   <xacro:azrael  prefix="$(arg prefix)">
@@ -64,5 +57,4 @@
     sim_ignition="$(arg sim_ignition)"
     headless_mode="$(arg headless_mode)"
-    initial_positions="${xacro.load_yaml(initial_positions_file)}"
     use_tool_communication="$(arg use_tool_communication)"
     tool_voltage="$(arg tool_voltage)"
@@ -75,7 +67,4 @@
     tool_tcp_port="$(arg tool_tcp_port)"
     robot_ip="$(arg robot_ip)"
-    script_filename="$(arg script_filename)"
-    output_recipe_filename="$(arg output_recipe_filename)"
-    input_recipe_filename="$(arg input_recipe_filename)"
     >
     <origin xyz="0 0 0" rpy="0 0 0" />
@@ -84,5 +73,5 @@
     <parent link="$(arg prefix)base_footprint"/>
     <child link="$(arg prefix)base_link"/>
-    <origin xyz="0 0 0.28" rpy=" 0 0 0"/>
+    <origin xyz="0.1 0 0.28" rpy=" 0 0 ${-M_PI/2}"/>
     <axis xyz="0 0 1"/>
   </joint>

Commit message: fix description

File: azrael_description/urdf/azrael/azrael.xacro (robot description, xacro)
@@ -17,5 +17,5 @@
     <link name="${prefix}base_link_azrael">
       <visual>
-        <origin xyz="0 0 0.032" rpy="0 0 -${M_PI/2}" />
+        <origin xyz="0 0 0.032" rpy="0 0 0" />
         <geometry>
           <mesh filename="file://$(find azrael_description)//meshes/azrael/visual/azrael.dae"/>
@@ -26,5 +26,5 @@
       </visual>
       <collision>
-        <origin xyz="0 0 0.032" rpy="0 0 -${M_PI/2}" />
+        <origin xyz="0 0 0.032" rpy="0 0 0" />
         <geometry>
           <mesh filename="file://$(find azrael_description)//meshes/azrael/collision/azrael.dae"/>
@@ -46,6 +46,5 @@
     <link name="${prefix}laser" />
     <joint name="${prefix}laser_joint" type="fixed">
-      <!-- <origin xyz="0.0 -0.65 0.3" rpy="0 0 -${M_PI/2}" /> -->
-      <origin xyz="0.65 0.0 0.3" rpy="0 0 0" />
+      <origin xyz="0.0 0.65 0.3" rpy="0 0 ${M_PI/2}" />
       <parent link="${prefix}base_link_azrael" />
       <child link="${prefix}laser" />

File: azrael_description/urdf/system.urdf.xacro (robot description, xacro)
@@ -73,5 +73,5 @@
     <parent link="$(arg prefix)base_footprint"/>
     <child link="$(arg prefix)base_link"/>
-    <origin xyz="0.1 0 0.28" rpy=" 0 0 ${-M_PI/2}"/>
+    <origin xyz="0.0 0.1 0.28" rpy=" 0 0 0"/>
     <axis xyz="0 0 1"/>
   </joint>

Commit message: ur changed

File: azrael_description/urdf/azrael/azrael.xacro (robot description, xacro)
@@ -19,5 +19,5 @@
         <origin xyz="0 0 0.032" rpy="0 0 0" />
         <geometry>
-          <mesh filename="file://$(find azrael_description)//meshes/azrael/visual/azrael.dae"/>
+          <mesh filename="file://$(find azrael_description)/meshes/azrael/visual/azrael.dae"/>
         </geometry>
         <material name="Gray">
@@ -28,5 +28,5 @@
         <origin xyz="0 0 0.032" rpy="0 0 0" />
         <geometry>
-          <mesh filename="file://$(find azrael_description)//meshes/azrael/collision/azrael.dae"/>
+          <mesh filename="file://$(find azrael_description)/meshes/azrael/collision/azrael.dae"/>
         </geometry>
         <material name="Gray">

File: azrael_description/urdf/system.urdf.xacro (robot description, xacro)
@@ -14,7 +14,7 @@
   </material>
   <xacro:include filename="$(find azrael_description)/urdf/azrael/azrael.xacro" />
+  <xacro:include filename="$(find ur_description)/urdf/ur_macro.xacro"/>
   <xacro:arg name="name" default="ur"/>
-  <xacro:include filename="$(find azrael_description)/urdf/ur_macro.xacro"/>
-  <xacro:arg name="ur_type" default="ur10"/>
+  <xacro:arg name="ur_type" default="ur10e"/>
   <!-- parameters -->
   <xacro:arg name="prefix" default="azrael/" />
@@ -23,4 +23,9 @@
   <xacro:arg name="physical_params" default="$(find azrael_description)/config/$(arg ur_type)/physical_parameters.yaml"/>
   <xacro:arg name="visual_params" default="$(find azrael_description)/config/$(arg ur_type)/visual_parameters.yaml"/>
+  <!-- <xacro:arg name="joint_limit_params" default="$(find ur_description)/config/ur10e/joint_limits.yaml"/>
+  <xacro:arg name="kinematics_params" default="$(find ur_description)/config/ur10e/default_kinematics.yaml"/>
+  <xacro:arg name="physical_params" default="$(find ur_description)/config/ur10e/physical_parameters.yaml"/>
+  <xacro:arg name="visual_params" default="$(find ur_description)/config/ur10e/visual_parameters.yaml"/>
+   -->
   <xacro:arg name="transmission_hw_interface" default=""/>
   <xacro:arg name="safety_limits" default="false"/>
@@ -29,5 +34,5 @@
   <!-- ros2_control related parameters -->
   <xacro:arg name="headless_mode" default="false" />
-  <xacro:arg name="robot_ip" default="0.0.0.0" />
+  <xacro:arg name="robot_ip" default="192.168.254.31" />
   <!--   tool communication related parameters-->
   <xacro:arg name="use_tool_communication" default="false" />
@@ -41,9 +46,20 @@
   <xacro:arg name="tool_tcp_port" default="54321" />
     <!-- Simulation parameters -->
-  <xacro:arg name="use_fake_hardware" default="false" />
-  <xacro:arg name="fake_sensor_commands" default="false" />
+  <xacro:arg name="fake_ur" default="true" />
+  <xacro:arg name="fake_sensor_commands" default="true" />
   <xacro:arg name="sim_gazebo" default="false" />
   <xacro:arg name="sim_ignition" default="false" />
   <xacro:arg name="simulation_controllers" default="error_default" />
+  <xacro:arg name="generate_ros2_control_tag" default="true" />
+  <xacro:arg name="script_filename" default="$(find ur_client_library)/resources/external_control.urscript" />
+  <xacro:arg name="output_recipe_filename" default="$(find ur_robot_driver)/resources/rtde_input_recipe.txt" />
+  <xacro:arg name="input_recipe_filename" default="$(find ur_robot_driver)/resources/rtde_output_recipe.txt" />
+  <xacro:arg name="reverse_port" default="50001" />
+  <xacro:arg name="script_sender_port" default="50002" />
+  <xacro:arg name="reverse_ip" default="0.0.0.0" />
+  <xacro:arg name="script_command_port" default="50004" />
+  <xacro:arg name="trajectory_port" default="50003" />
+  <xacro:arg name="non_blocking_read" default="true" />
+  <xacro:arg name="keep_alive_count" default="2" />
   <xacro:property name="M_PI" value="3.14159"/>
   <xacro:azrael  prefix="$(arg prefix)">
@@ -51,8 +67,8 @@
   </xacro:azrael>
   <!-- <link name="$(arg prefix)base_footprint"/> -->
-   <!-- arm -->
+  <!-- new arm -->
   <xacro:ur_robot
     name="$(arg name)"
-    prefix="$(arg prefix)"
+    tf_prefix="$(arg prefix)"
     parent="$(arg prefix)base_footprint"
     joint_limits_parameters_file="$(arg joint_limit_params)"
@@ -60,14 +76,15 @@
     physical_parameters_file="$(arg physical_params)"
     visual_parameters_file="$(arg visual_params)"
-    initial_positions="${dict(shoulder_pan_joint=1.0,shoulder_lift_joint=-2.30,elbow_joint=2.26,wrist_1_joint=-0.43,wrist_2_joint=0.75,wrist_3_joint=0.0)}"
-    transmission_hw_interface="$(arg transmission_hw_interface)"
     safety_limits="$(arg safety_limits)"
     safety_pos_margin="$(arg safety_pos_margin)"
     safety_k_position="$(arg safety_k_position)"
-    use_fake_hardware="$(arg use_fake_hardware)"
+    use_fake_hardware="$(arg fake_ur)"
+    generate_ros2_control_tag="$(arg generate_ros2_control_tag)"
+    transmission_hw_interface="$(arg transmission_hw_interface)"
     fake_sensor_commands="$(arg fake_sensor_commands)"
     sim_gazebo="$(arg sim_gazebo)"
     sim_ignition="$(arg sim_ignition)"
     headless_mode="$(arg headless_mode)"
+    initial_positions="${dict(shoulder_pan_joint=1.0,shoulder_lift_joint=-2.30,elbow_joint=2.26,wrist_1_joint=-0.43,wrist_2_joint=0.75,wrist_3_joint=0.0)}"
     use_tool_communication="$(arg use_tool_communication)"
     tool_voltage="$(arg tool_voltage)"
@@ -80,8 +97,16 @@
     tool_tcp_port="$(arg tool_tcp_port)"
     robot_ip="$(arg robot_ip)"
-    >
-    <origin xyz="0.0 0.1 0.28" rpy="0 0 0"/>
-<!--    <origin xyz="0.0 0.0 0.28" rpy="0 0 0"/>-->
-  </xacro:ur_robot>
+    script_filename="$(arg script_filename)"
+    output_recipe_filename="$(arg output_recipe_filename)"
+    input_recipe_filename="$(arg input_recipe_filename)"
+    reverse_port="$(arg reverse_port)"
+    script_sender_port="$(arg script_sender_port)"
+    reverse_ip="$(arg reverse_ip)"
+    script_command_port="$(arg script_command_port)"
+    trajectory_port="$(arg trajectory_port)"
+    non_blocking_read="$(arg non_blocking_read)"
+    keep_alive_count="$(arg keep_alive_count)">
+    <origin xyz="0.0 0.1 0.28" rpy="0 0 0" />          <!-- position robot in the world -->
+   </xacro:ur_robot>
 <!--  <link name="$(arg prefix)tcp" />
   <joint name="$(arg prefix)tcpjoint" type="fixed">

File: azrael_description/urdf/ur_common.xacro (robot description, xacro)
@@ -40,11 +40,11 @@
     <xacro:property name="force_abs_paths" value="${force_abs_paths}" scope="parent"/>
     <!-- Read .yaml files from disk, load content into properties -->
-    <xacro:property name="config_joint_limit_parameters" value="${load_yaml(joint_limits_parameters_file)}"/>
-    <xacro:property name="config_kinematics_parameters" value="${load_yaml(kinematics_parameters_file)}"/>
-    <xacro:property name="config_physical_parameters" value="${load_yaml(physical_parameters_file)}"/>
-    <xacro:property name="config_visual_parameters" value="${load_yaml(visual_parameters_file)}"/>
+    <xacro:property name="config_joint_limit_parameters" value="${xacro.load_yaml(joint_limits_parameters_file)}"/>
+    <xacro:property name="config_kinematics_parameters" value="${xacro.load_yaml(kinematics_parameters_file)}"/>
+    <xacro:property name="config_physical_parameters" value="${xacro.load_yaml(physical_parameters_file)}"/>
+    <xacro:property name="config_visual_parameters" value="${xacro.load_yaml(visual_parameters_file)}"/>
     <!-- Extract subsections from yaml dictionaries -->
     <xacro:property name="sec_limits" value="${config_joint_limit_parameters['joint_limits']}"/>
-    <xacro:property name="sec_dh_parameters" value="${config_physical_parameters['dh_parameters']}"/>
+    <!-- <xacro:property name="sec_dh_parameters" value="${config_physical_parameters['dh_parameters']}"/> -->
     <xacro:property name="sec_offsets" value="${config_physical_parameters['offsets']}"/>
     <xacro:property name="sec_inertia_parameters" value="${config_physical_parameters['inertia_parameters']}" />
@@ -77,10 +77,10 @@
     <xacro:property name="wrist_3_effort_limit" value="${sec_limits['wrist_3_joint']['max_effort']}" scope="parent"/>
     <!-- DH PARAMETERS -->
-    <xacro:property name="d1" value="${sec_dh_parameters['d1']}" scope="parent"/>
+    <!-- <xacro:property name="d1" value="${sec_dh_parameters['d1']}" scope="parent"/>
     <xacro:property name="a2" value="${sec_dh_parameters['a2']}" scope="parent"/>
     <xacro:property name="a3" value="${sec_dh_parameters['a3']}" scope="parent"/>
     <xacro:property name="d4" value="${sec_dh_parameters['d4']}" scope="parent"/>
     <xacro:property name="d5" value="${sec_dh_parameters['d5']}" scope="parent"/>
-    <xacro:property name="d6" value="${sec_dh_parameters['d6']}" scope="parent"/>
+    <xacro:property name="d6" value="${sec_dh_parameters['d6']}" scope="parent"/> -->
     <!-- kinematics -->
     <xacro:property name="shoulder_x" value="${sec_kinematics['shoulder']['x']}" scope="parent"/>

Commit message: force_torque_sensor_controller

File: azrael_description/urdf/azrael/azrael.xacro (robot description, xacro)
@@ -19,4 +19,5 @@
         <origin xyz="0 0 0.032" rpy="0 0 0" />
         <geometry>
+          <!-- <mesh filename="package://azrael_description/meshes/azrael/visual/azrael.dae"/> -->
           <mesh filename="file://$(find azrael_description)/meshes/azrael/visual/azrael.dae"/>
         </geometry>

Commit message: base footprint rotated

File: azrael_description/urdf/azrael/azrael.xacro (robot description, xacro)
@@ -44,4 +44,5 @@
       <parent link="${prefix}base_footprint" />
       <child link="${prefix}base_link_azrael" />
+      <origin xyz="0 0 0.0" rpy="0 0 -${M_PI/2}" />
     </joint>
     <link name="${prefix}laser" />

File: azrael_description/urdf/ur_macro.xacro (robot description, xacro)
@@ -199,4 +199,5 @@
       <parent link="${parent}" />
       <child link="${prefix}base_link" />
+      <origin xyz="0 0 0" rpy="0 0 -${pi}" />
     </joint>
     <!-- joints - main serial chain -->

Commit message: test

File: azrael_description/urdf/azrael/azrael.xacro (robot description, xacro)
@@ -44,5 +44,5 @@
       <parent link="${prefix}base_footprint" />
       <child link="${prefix}base_link_azrael" />
-      <origin xyz="0 0 0.0" rpy="0 0 -${M_PI/2}" />
+      <!-- <origin xyz="0 0 0.0" rpy="0 0 -${M_PI/2}" /> -->
     </joint>
     <link name="${prefix}laser" />

Commit message: Nav2 param

File: azrael_description/urdf/azrael/azrael.xacro (robot description, xacro)
@@ -44,5 +44,4 @@
       <parent link="${prefix}base_footprint" />
       <child link="${prefix}base_link_azrael" />
-      <!-- <origin xyz="0 0 0.0" rpy="0 0 -${M_PI/2}" /> -->
     </joint>
     <link name="${prefix}laser" />

Commit message: Several changes: cnr admittance, robot localization

File: azrael_description/urdf/azrael/azrael.xacro (robot description, xacro)
@@ -20,5 +20,5 @@
         <geometry>
           <!-- <mesh filename="package://azrael_description/meshes/azrael/visual/azrael.dae"/> -->
-          <mesh filename="file://$(find azrael_description)/meshes/azrael/visual/azrael.dae"/>
+          <mesh filename="package://azrael_description/meshes/azrael/visual/azrael.dae"/>
         </geometry>
         <material name="Gray">
@@ -29,5 +29,5 @@
         <origin xyz="0 0 0.032" rpy="0 0 0" />
         <geometry>
-          <mesh filename="file://$(find azrael_description)/meshes/azrael/collision/azrael.dae"/>
+          <mesh filename="package://azrael_description/meshes/azrael/collision/azrael.dae"/>
         </geometry>
         <material name="Gray">

Commit message: * add wheel publisher * change mesh url

File: azrael_description/urdf/azrael/azrael.xacro (robot description, xacro)
@@ -19,6 +19,6 @@
         <origin xyz="0 0 0.032" rpy="0 0 0" />
         <geometry>
-          <!-- <mesh filename="package://azrael_description/meshes/azrael/visual/azrael.dae"/> -->
-          <mesh filename="file://$(find azrael_description)/meshes/azrael/visual/azrael.dae"/>
+          <mesh filename="package://azrael_description/meshes/azrael/visual/azrael.dae"/>
+          <!-- <mesh filename="file://$(find azrael_description)/meshes/azrael/visual/azrael.dae"/> -->
         </geometry>
         <material name="Gray">
@@ -29,5 +29,6 @@
         <origin xyz="0 0 0.032" rpy="0 0 0" />
         <geometry>
-          <mesh filename="file://$(find azrael_description)/meshes/azrael/collision/azrael.dae"/>
+          <!-- <mesh filename="file://$(find azrael_description)/meshes/azrael/collision/azrael.dae"/> -->
+          <mesh filename="package://azrael_description/meshes/azrael/collision/azrael.dae"/>
         </geometry>
         <material name="Gray">
