Commit message: Split base and arm, with two state publishers

File: azrael_description/urdf/azrael/azrael_base.xacro (robot description, xacro)
@@ -6,5 +6,5 @@
   <xacro:property name="base_y_size" value="0.55" />
   <xacro:property name="base_z_size" value="0.35" />
-  <xacro:macro name="azrael" params="prefix *origin">
+  <xacro:macro name="azrael_base" params="prefix *origin">
     <!-- Base footprint is on the ground under the robot -->
     <link name="${prefix}base_footprint">

File: azrael_description/urdf/azrael_arm.urdf.xacro (robot description, xacro)
@@ -1,5 +1,4 @@
 <?xml version="1.0"?>
-<robot name="azrael" xmlns:xacro="http://ros.org/wiki/xacro">
-  <xacro:include filename="azrael/azrael_base.xacro"/>
+<robot name="azrael_arm" xmlns:xacro="http://ros.org/wiki/xacro">
   <xacro:include filename="azrael/azrael_arm.xacro"/>
   <xacro:arg name="name" default="ur"/>
@@ -31,5 +30,5 @@
   <xacro:arg name="sim_gazebo" default="false"/>
   <xacro:arg name="sim_ignition" default="false"/>
-  <xacro:arg name="generate_ros2_control_tag" default="true"/>
+  <xacro:arg name="generate_ros2_control_tag" default="false"/>
   <xacro:arg name="script_filename" default="$(find ur_client_library)/resources/external_control.urscript"/>
   <xacro:arg name="output_recipe_filename" default="$(find ur_robot_driver)/resources/rtde_output_recipe.txt"/>
@@ -42,8 +41,5 @@
   <xacro:arg name="non_blocking_read" default="true"/>
   <xacro:arg name="keep_alive_count" default="2"/>
-  <xacro:property name="M_PI" value="3.14159"/>
-  <xacro:azrael_base prefix="$(arg prefix)">
-    <origin xyz="0 0 0" rpy="0 0 -${M_PI/2}"/>
-  </xacro:azrael_base>
+  <link name="$(arg prefix)base_footprint"/>
   <xacro:azrael_arm parent="$(arg prefix)base_footprint"/>
 </robot>
